Commit message: created script to convert ptx to pcd file

File: urdf/camera.urdf.xacro (robot description, xacro)
@@ -19,5 +19,5 @@
             <origin xyz="$(arg x) $(arg y) $(arg z)"/>
             <geometry>
-                <mesh filename="file:///$(find gazebo_simulation)/meshes/asus_xtion.dae"/>
+                <mesh filename="file:///$(find leica_scanstation)/meshes/asus_xtion.dae"/>
             </geometry>
         </collision>
