Commit message: new part scale

File: urdf/assembly_big.xacro (robot description, xacro)
@@ -13,5 +13,5 @@
             <origin xyz="$(arg x) $(arg y) $(arg z)"/>
             <geometry>
-                <mesh filename="file:///$(find leica_scanstation)/meshes/Assembly2.dae" scale="0.001 0.001 0.001"/>
+                <mesh filename="file:///$(find leica_scanstation)/meshes/Assembly2.dae" scale="0.0005 0.0005 0.0005"/>
             </geometry>
         </visual>
@@ -19,5 +19,5 @@
             <origin xyz="$(arg x) $(arg y) $(arg z)"/>
             <geometry>
-                <mesh filename="file:///$(find leica_scanstation)/meshes/Assembly2.dae" scale="0.001 0.001 0.001"/>
+                <mesh filename="file:///$(find leica_scanstation)/meshes/Assembly2.dae" scale="0.0005 0.0005 0.0005"/>
             </geometry>
         </collision>

Commit message: minor changes related to gazebo

File: urdf/assembly_big.xacro (robot description, xacro)
@@ -13,5 +13,6 @@
             <origin xyz="$(arg x) $(arg y) $(arg z)"/>
             <geometry>
-                <mesh filename="file:///$(find leica_scanstation)/meshes/Assembly2.dae" scale="0.0005 0.0005 0.0005"/>
+                <!-- <mesh filename="file:///$(find leica_scanstation)/meshes/Assembly2.dae" scale="0.0005 0.0005 0.0005"/> -->
+                <mesh filename="file:///$(find leica_scanstation)/meshes/untitled.obj"/>
             </geometry>
         </visual>
@@ -19,5 +20,5 @@
             <origin xyz="$(arg x) $(arg y) $(arg z)"/>
             <geometry>
-                <mesh filename="file:///$(find leica_scanstation)/meshes/Assembly2.dae" scale="0.0005 0.0005 0.0005"/>
+                <mesh filename="file:///$(find leica_scanstation)/meshes/untitled.obj"/>
             </geometry>
         </collision>

File: urdf/camera.urdf.xacro (robot description, xacro)
@@ -34,15 +34,15 @@
                 <scan>
                     <horizontal>
-                        <samples>20</samples>
+                        <samples>520</samples>
                         <resolution>1</resolution>
                         <min_angle>-1.57</min_angle>
                         <max_angle>1.57</max_angle>
                     </horizontal>
-                    <vertical>
+                    <!-- <vertical>
                         <samples>520</samples>
                         <resolution>1</resolution>
                         <min_angle>-1.57</min_angle>
                         <max_angle>1.57</max_angle>
-                    </vertical>
+                    </vertical> -->
                 </scan>
                 <range>
